File: EurorackPower.kicad_sch (KiCad schematic)
At the start: 16 parts, among them J1 europower, J2 Conn_01x02, J3 Conn_01x03, J4 Conn_01x02, J5 Conn_01x03

Commit message: bom and schematic
Parts:
- H1, H2: now left out of the parts list
Changed lines of the file:
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@@
   )
   (symbol (lib_id "Mechanical:MountingHole") (at 127 114.3 0) (unit 1)
-    (in_bom yes) (on_board yes) (fields_autoplaced)
+    (in_bom no) (on_board yes) (fields_autoplaced)
     (property "Reference" "H1" (id 0) (at 130.048 113.0299 0)
       (effects (font (size 1.27 1.27)) (justify left))
@@
   )
   (symbol (lib_id "Mechanical:MountingHole") (at 152.4 114.3 0) (unit 1)
-    (in_bom yes) (on_board yes) (fields_autoplaced)
+    (in_bom no) (on_board yes) (fields_autoplaced)
     (property "Reference" "H2" (id 0) (at 155.448 113.0299 0)
       (effects (font (size 1.27 1.27)) (justify left))
